File: hardware/fireflycap.sch (KiCad schematic (older format))
At the start: 58 parts, among them P1 CONN_1, P10 CONN_2X2, P11 CONN_2, P12 CONN_1, P13 CONN_2, P14 JTAG, P15 CONN_2, P16 CONN_1, P17 CONN_2, P18 CONN_2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

Commit message: bom corrections
Parts:
- C1: Part Number ESHR-0003C0-002R7 -> ESHSR-0003C0-002R7
- R10: Description Thick Film Resistors Thick Film Chip Res 0603 1/16W 5% -> RES 330 OHM 1/10W 5% 0603 SMD; Part Number ERJ-3GEYJ101V -> ERJ-3GEYJ331V
Changed lines of the file:
@@
-EESchema Schematic File Version 2  date Thu May  3 22:59:48 2012
+EESchema Schematic File Version 2  date Mon May  7 21:24:55 2012
 LIBS:fireflycap
 LIBS:power
@@
 Sheet 1 1
 Title "Firefly Cap"
-Date "3 may 2012"
+Date "8 may 2012"
 Rev ""
 Comp "Copyright 2012 Michael Ossmann"
@@
 F 2 "GSG-0603" H 7550 2700 60  0001 C CNN
 F 4 "Panasonic" V 7550 2700 60  0001 C CNN "Manufacturer"
-F 5 "ERJ-3GEYJ101V" V 7550 2700 60  0001 C CNN "Part Number"
-F 6 "Thick Film Resistors Thick Film Chip Res 0603 1/16W 5%" V 7550 2700 60  0001 C CNN "Description"
+F 5 "ERJ-3GEYJ331V" V 7550 2700 60  0001 C CNN "Part Number"
+F 6 "RES 330 OHM 1/10W 5% 0603 SMD" V 7550 2700 60  0001 C CNN "Description"
 	1    7550 2700
 	-1   0    0    1
@@
 F 2 "GSG-ESHSR-0003-SIDE" H 1750 2200 60  0001 C CNN
 F 4 "Nesscap" H 1750 2200 60  0001 C CNN "Manufacturer"
-F 5 "ESHR-0003C0-002R7" H 1750 2200 60  0001 C CNN "Part Number"
+F 5 "ESHSR-0003C0-002R7" H 1750 2200 60  0001 C CNN "Part Number"
 F 6 "Ultracapacitor 3F 2.7V" H 1750 2200 60  0001 C CNN "Description"
 	1    1750 2200

Commit message: filled in bom info for some passives
Parts:
- C4: Description (none) -> CAP CER 2200PF 50V 20% X7R 0603; Manufacturer (none) -> Murata; Part Number (none) -> GRM188R71H222MA01D
- C7, C8: Description (none) -> CAP CER 2200PF 50V 10% X7R 0805; Manufacturer (none) -> Kemet; Part Number (none) -> C0805C222K5RACTU
- R1: Description (none) -> RES 47K OHM 1/10W 5% 0603 SMD; Manufacturer (none) -> Panasonic; Part Number (none) -> ERJ-3GEYJ473V
- R11, R13, R14: Description (none) -> RES 4.7M OHM 1/8W 5% 0805 SMD; Manufacturer (none) -> Panasonic; Part Number (none) -> ERJ-6GEYJ475V
- R12, R15, R16, R17, R18: Description (none) -> RESISTOR 10M OHM 1/8W 5% 0805; Manufacturer (none) -> Panasonic; Part Number (none) -> ERJ-6GEYJ106V
- R2, R3, R8, R9: Description (none) -> RES 4.70M OHM 1/8W 1% 0805 SMD; Manufacturer (none) -> Vishay Dale; Part Number (none) -> CRCW08054M70FKEA
Changed lines of the file:
@@
-EESchema Schematic File Version 2  date Mon May  7 21:24:55 2012
+EESchema Schematic File Version 2  date Wed May  9 18:00:23 2012
 LIBS:fireflycap
 LIBS:power
@@
 Sheet 1 1
 Title "Firefly Cap"
-Date "8 may 2012"
+Date "10 may 2012"
 Rev ""
 Comp "Copyright 2012 Michael Ossmann"
@@
 F 1 "4M7" V 5900 5950 50  0000 C CNN
 F 2 "GSG-0805" H 5900 5950 60  0001 C CNN
+F 4 "Panasonic" H 5900 5950 60  0001 C CNN "Manufacturer"
+F 5 "ERJ-6GEYJ475V" H 5900 5950 60  0001 C CNN "Part Number"
+F 6 "RES 4.7M OHM 1/8W 5% 0805 SMD" H 5900 5950 60  0001 C CNN "Description"
 	1    5900 5950
 	-1   0    0    1
@@
 F 1 "10M" V 5150 6600 50  0000 C CNN
 F 2 "GSG-0805" H 5150 6600 60  0001 C CNN
+F 4 "Panasonic" H 5150 6600 60  0001 C CNN "Manufacturer"
+F 5 "ERJ-6GEYJ106V" H 5150 6600 60  0001 C CNN "Part Number"
+F 6 "RESISTOR 10M OHM 1/8W 5% 0805" H 5150 6600 60  0001 C CNN "Description"
 	1    5150 6600
 	0    1    1    0
@@
 F 1 "10M" V 4800 6950 50  0000 C CNN
 F 2 "GSG-0805" H 4800 6950 60  0001 C CNN
+F 4 "Panasonic" H 4800 6950 60  0001 C CNN "Manufacturer"
+F 5 "ERJ-6GEYJ106V" H 4800 6950 60  0001 C CNN "Part Number"
+F 6 "RESISTOR 10M OHM 1/8W 5% 0805" H 4800 6950 60  0001 C CNN "Description"
 	1    4800 6950
 	1    0    0    -1
@@
 F 1 "4M7" V 2950 6600 50  0000 C CNN
 F 2 "GSG-0805" H 2950 6600 60  0001 C CNN
+F 4 "Panasonic" H 2950 6600 60  0001 C CNN "Manufacturer"
+F 5 "ERJ-6GEYJ475V" H 2950 6600 60  0001 C CNN "Part Number"
+F 6 "RES 4.7M OHM 1/8W 5% 0805 SMD" H 2950 6600 60  0001 C CNN "Description"
 	1    2950 6600
 	0    1    1    0
@@
 F 1 "10M" V 2600 6950 50  0000 C CNN
 F 2 "GSG-0805" H 2600 6950 60  0001 C CNN
+F 4 "Panasonic" H 2600 6950 60  0001 C CNN "Manufacturer"
+F 5 "ERJ-6GEYJ106V" H 2600 6950 60  0001 C CNN "Part Number"
+F 6 "RESISTOR 10M OHM 1/8W 5% 0805" H 2600 6950 60  0001 C CNN "Description"
 	1    2600 6950
 	1    0    0    -1
@@
 F 1 "4M7" V 3950 6300 50  0000 C CNN
 F 2 "GSG-0805" H 3950 6300 60  0001 C CNN
+F 4 "Panasonic" H 3950 6300 60  0001 C CNN "Manufacturer"
+F 5 "ERJ-6GEYJ475V" H 3950 6300 60  0001 C CNN "Part Number"
+F 6 "RES 4.7M OHM 1/8W 5% 0805 SMD" H 3950 6300 60  0001 C CNN "Description"
 	1    3950 6300
 	0    1    1    0
@@
 F 1 "2.2nF" H 9550 1550 50  0000 L CNN
 F 2 "GSG-0805" H 9500 1650 60  0001 C CNN
+F 4 "Kemet" H 9500 1650 60  0001 C CNN "Manufacturer"
+F 5 "C0805C222K5RACTU" H 9500 1650 60  0001 C CNN "Part Number"
+F 6 "CAP CER 2200PF 50V 10% X7R 0805" H 9500 1650 60  0001 C CNN "Description"
 	1    9500 1650
 	1    0    0    1
@@
 F 1 "2.2nF" H 8150 1550 50  0000 L CNN
 F 2 "GSG-0805" H 8100 1650 60  0001 C CNN
+F 4 "Kemet" H 8100 1650 60  0001 C CNN "Manufacturer"
+F 5 "C0805C222K5RACTU" H 8100 1650 60  0001 C CNN "Part Number"
+F 6 "CAP CER 2200PF 50V 10% X7R 0805" H 8100 1650 60  0001 C CNN "Description"
 	1    8100 1650
 	-1   0    0    1
@@
 F 1 "10M" V 1650 6600 50  0000 C CNN
 F 2 "GSG-0805" H 1650 6600 60  0001 C CNN
+F 4 "Panasonic" H 1650 6600 60  0001 C CNN "Manufacturer"
+F 5 "ERJ-6GEYJ106V" H 1650 6600 60  0001 C CNN "Part Number"
+F 6 "RESISTOR 10M OHM 1/8W 5% 0805" H 1650 6600 60  0001 C CNN "Description"
 	1    1650 6600
 	0    1    1    0
@@
 F 1 "10M" V 2300 5950 50  0000 C CNN
 F 2 "GSG-0805" H 2300 5950 60  0001 C CNN
+F 4 "Panasonic" H 2300 5950 60  0001 C CNN "Manufacturer"
+F 5 "ERJ-6GEYJ106V" H 2300 5950 60  0001 C CNN "Part Number"
+F 6 "RESISTOR 10M OHM 1/8W 5% 0805" H 2300 5950 60  0001 C CNN "Description"
 	1    2300 5950
 	1    0    0    -1
@@
 F 1 "4M7" V 9200 1000 50  0000 C CNN
 F 2 "GSG-0805" H 9200 1000 60  0001 C CNN
+F 4 "Vishay Dale" H 9200 1000 60  0001 C CNN "Manufacturer"
+F 5 "CRCW08054M70FKEA" H 9200 1000 60  0001 C CNN "Part Number"
+F 6 "RES 4.70M OHM 1/8W 1% 0805 SMD" H 9200 1000 60  0001 C CNN "Description"
 	1    9200 1000
 	-1   0    0    1
@@
 F 1 "4M7" V 9200 1700 50  0000 C CNN
 F 2 "GSG-0805" H 9200 1700 60  0001 C CNN
+F 4 "Vishay Dale" H 9200 1700 60  0001 C CNN "Manufacturer"
+F 5 "CRCW08054M70FKEA" H 9200 1700 60  0001 C CNN "Part Number"
+F 6 "RES 4.70M OHM 1/8W 1% 0805 SMD" H 9200 1700 60  0001 C CNN "Description"
 	1    9200 1700
 	-1   0    0    1
@@
 F 1 "2.2nF" H 10250 3650 50  0000 L CNN
 F 2 "GSG-0603" H 10200 3750 60  0001 C CNN
+F 4 "Murata" H 10200 3750 60  0001 C CNN "Manufacturer"
+F 5 "GRM188R71H222MA01D" H 10200 3750 60  0001 C CNN "Part Number"
+F 6 "CAP CER 2200PF 50V 20% X7R 0603" H 10200 3750 60  0001 C CNN "Description"
 	1    10200 3750
 	-1   0    0    1
@@
 F 1 "4M7" V 8400 1700 50  0000 C CNN
 F 2 "GSG-0805" H 8400 1700 60  0001 C CNN
+F 4 "Vishay Dale" H 8400 1700 60  0001 C CNN "Manufacturer"
+F 5 "CRCW08054M70FKEA" H 8400 1700 60  0001 C CNN "Part Number"
+F 6 "RES 4.70M OHM 1/8W 1% 0805 SMD" H 8400 1700 60  0001 C CNN "Description"
 	1    8400 1700
 	-1   0    0    1
@@
 F 1 "4M7" V 8400 1000 50  0000 C CNN
 F 2 "GSG-0805" H 8400 1000 60  0001 C CNN
+F 4 "Vishay Dale" H 8400 1000 60  0001 C CNN "Manufacturer"
+F 5 "CRCW08054M70FKEA" H 8400 1000 60  0001 C CNN "Part Number"
+F 6 "RES 4.70M OHM 1/8W 1% 0805 SMD" H 8400 1000 60  0001 C CNN "Description"
 	1    8400 1000
 	-1   0    0    1
@@
 F 1 "47k" V 10200 3100 50  0000 C CNN
 F 2 "GSG-0603" H 10200 3100 60  0001 C CNN
+F 4 "Panasonic" H 10200 3100 60  0001 C CNN "Manufacturer"
+F 5 "ERJ-3GEYJ473V" H 10200 3100 60  0001 C CNN "Part Number"
+F 6 "RES 47K OHM 1/10W 5% 0603 SMD" H 10200 3100 60  0001 C CNN "Description"
 	1    10200 3100
 	1    0    0    -1
